File: pcb/OK35.kicad_sch (KiCad schematic)
At the start: 74 parts, among them SW1 SW_SPST, SW10 SW_SPST, SW11 SW_SPST, SW12 SW_SPST, SW13 SW_SPST, SW14 SW_SPST, SW15 SW_SPST, SW16 SW_SPST, SW17 SW_SPST, SW18 SW_SPST, SW19 SW_SPST, SW2 SW_SPST, SW20 SW_SPST, SW21 SW_SPST, SW22 SW_SPST, SW23 SW_SPST, SW24 SW_SPST, SW25 SW_SPST, SW26 SW_SPST, SW27 SW_SPST, SW28 SW_SPST, SW29 SW_SPST, SW3 SW_SPST, SW30 SW_SPST, SW31 SW_SPST, SW32 SW_SPST, SW33 SW_SPST, SW34 SW_SPST, SW35 SW_SPST, SW4 SW_SPST, SW5 SW_SPST, SW6 SW_SPST, SW7 SW_SPST, SW8 SW_SPST, SW9 SW_SPST, U1 TRRS, U2 ProMicro

Commit message: v0.1.2 - add handedness jumper
Parts:
- added JP1: SolderJumper_3_Open, Jumper:SolderJumper-3_P2.0mm_Open_TrianglePad1.0x1.5mm, symbol Jumper:SolderJumper_3_Open
Connections:
- net GND: now also JP1.3 (B)
- net VCC: now also JP1.1 (A)
- net at U2.20 (A3/PF4): now also JP1.2 (C)
Changed lines of the file:
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@@
+    (stroke (width 0) (type default) (color 0 0 0 0))
+  )
+  (wire (pts (xy 119.38 93.98) (xy 127 93.98))
     (stroke (width 0) (type default) (color 0 0 0 0))
   )
@@
     (pin "1")
   )
+  (symbol (lib_id "power:VCC") (at 130.81 88.9 0) (unit 1)
+    (in_bom yes) (on_board yes) (fields_autoplaced)
+    (property "Reference" "#PWR0101" (id 0) (at 130.81 92.71 0)
+      (effects (font (size 1.27 1.27)) hide)
+    )
+    (property "Value" "VCC" (id 1) (at 130.81 85.3242 0))
+    (property "Footprint" "" (id 2) (at 130.81 88.9 0)
+      (effects (font (size 1.27 1.27)) hide)
+    )
+    (property "Datasheet" "" (id 3) (at 130.81 88.9 0)
+      (effects (font (size 1.27 1.27)) hide)
+    )
+    (pin "1")
+  )
   (symbol (lib_id "Device:D") (at 213.36 54.61 90) (unit 1)
     (in_bom yes) (on_board yes) (fields_autoplaced)
@@
     (pin "1")
     (pin "2")
+  )
+  (symbol (lib_id "Jumper:SolderJumper_3_Open") (at 130.81 93.98 270) (unit 1)
+    (in_bom yes) (on_board yes) (fields_autoplaced)
+    (property "Reference" "JP1" (id 0) (at 132.461 94.4138 90)
+      (effects (font (size 1.27 1.27)) (justify left))
+    )
+    (property "Value" "SolderJumper_3_Open" (id 1) (at 132.461 95.6822 90)
+      (effects (font (size 1.27 1.27)) (justify left) hide)
+    )
+    (property "Footprint" "Jumper:SolderJumper-3_P2.0mm_Open_TrianglePad1.0x1.5mm" (id 2) (at 130.81 93.98 0)
+      (effects (font (size 1.27 1.27)) hide)
+    )
+    (property "Datasheet" "~" (id 3) (at 130.81 93.98 0)
+      (effects (font (size 1.27 1.27)) hide)
+    )
+    (pin "1")
+    (pin "2")
+    (pin "3")
   )
   (symbol (lib_id "Switch:SW_SPST") (at 182.88 88.9 0) (unit 1)
@@
     (pin "1")
     (pin "2")
+  )
+  (symbol (lib_id "power:GND") (at 130.81 99.06 0) (unit 1)
+    (in_bom yes) (on_board yes) (fields_autoplaced)
+    (property "Reference" "#PWR0102" (id 0) (at 130.81 105.41 0)
+      (effects (font (size 1.27 1.27)) hide)
+    )
+    (property "Value" "GND" (id 1) (at 130.81 103.5034 0))
+    (property "Footprint" "" (id 2) (at 130.81 99.06 0)
+      (effects (font (size 1.27 1.27)) hide)
+    )
+    (property "Datasheet" "" (id 3) (at 130.81 99.06 0)
+      (effects (font (size 1.27 1.27)) hide)
+    )
+    (pin "1")
   )
   (symbol (lib_id "Switch:SW_SPST") (at 157.48 50.8 0) (unit 1)
@@
       (reference "#PWR08") (unit 1) (value "VCC") (footprint "")
     )
+    (path "/563758b7-ae21-4c67-9f90-29a86ae6265d"
+      (reference "#PWR0101") (unit 1) (value "VCC") (footprint "")
+    )
+    (path "/a280521c-c74b-4ecf-b9b4-213ba488c164"
+      (reference "#PWR0102") (unit 1) (value "GND") (footprint "")
+    )
     (path "/01c7a84d-d1ee-4603-ac37-663df33343ae"
       (reference "D1") (unit 1) (value "D") (footprint "keebio:MD_Diode")
@@
       (reference "D35") (unit 1) (value "D") (footprint "keebio:MD_Diode")
     )
+    (path "/738c73ca-416f-4cdc-b135-180d4d696484"
+      (reference "JP1") (unit 1) (value "SolderJumper_3_Open") (footprint "Jumper:SolderJumper-3_P2.0mm_Open_TrianglePad1.0x1.5mm")
+    )
     (path "/37e9bfa6-9f52-4e15-b12d-0781db7a2c82"

Commit message: v0.1.3 - standard 2u switch options
Parts:
- added SW36, SW37: SW_SPST, keebio:MX-Alps-Choc-2U, symbol Switch:SW_SPST
Connections:
- net Col1: now also SW36.1 (A)
- net Col5: now also SW37.1 (A)
- net at D30.2 (A), SW30.2 (B): now also SW36.2 (B)
- net at D34.2 (A), SW34.2 (B): now also SW37.2 (B)
Changed lines of the file:
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@@
   (title_block
     (title "OK35")
-    (date "2022-02-21")
-    (rev "0.1.1")
+    (date "2022-03-06")
+    (rev "0.1.3")
     (company "moth.monster")
   )
@@
   (junction (at 200.66 109.22) (diameter 0) (color 0 0 0 0)
   )
+  (junction (at 162.56 101.6) (diameter 0) (color 0 0 0 0)
+  )
   (junction (at 200.66 71.12) (diameter 0) (color 0 0 0 0)
   )
@@
   (junction (at 226.06 109.22) (diameter 0) (color 0 0 0 0)
   )
+  (junction (at 203.2 100.33) (diameter 0) (color 0 0 0 0)
+  )
   (junction (at 190.5 88.9) (diameter 0) (color 0 0 0 0)
   )
@@
   (junction (at 187.96 83.82) (diameter 0) (color 0 0 0 0)
   )
+  (junction (at 213.36 101.6) (diameter 0) (color 0 0 0 0)
+  )
   (junction (at 215.9 63.5) (diameter 0) (color 0 0 0 0)
   )
+  (junction (at 152.4 100.33) (diameter 0) (color 0 0 0 0)
+  )
   (junction (at 190.5 76.2) (diameter 0) (color 0 0 0 0)
   )
@@
     (stroke (width 0) (type default) (color 0 0 0 0))
   )
-  (wire (pts (xy 152.4 88.9) (xy 152.4 101.6))
+  (wire (pts (xy 152.4 88.9) (xy 152.4 100.33))
     (stroke (width 0) (type default) (color 0 0 0 0))
   )
@@
     (stroke (width 0) (type default) (color 0 0 0 0))
   )
+  (wire (pts (xy 190.5 88.9) (xy 190.5 101.6))
+    (stroke (width 0) (type default) (color 0 0 0 0))
+  )
   (wire (pts (xy 139.7 88.9) (xy 139.7 101.6))
     (stroke (width 0) (type default) (color 0 0 0 0))
   )
-  (wire (pts (xy 190.5 88.9) (xy 190.5 101.6))
-    (stroke (width 0) (type default) (color 0 0 0 0))
-  )
   (wire (pts (xy 200.66 83.82) (xy 213.36 83.82))
     (stroke (width 0) (type default) (color 0 0 0 0))
@@
     (stroke (width 0) (type default) (color 0 0 0 0))
   )
-  (wire (pts (xy 203.2 88.9) (xy 203.2 101.6))
+  (wire (pts (xy 203.2 88.9) (xy 203.2 100.33))
     (stroke (width 0) (type default) (color 0 0 0 0))
   )
@@
     (stroke (width 0) (type default) (color 0 0 0 0))
   )
+  (wire (pts (xy 213.36 100.33) (xy 213.36 101.6))
+    (stroke (width 0) (type default) (color 0 0 0 0))
+  )
   (wire (pts (xy 215.9 50.8) (xy 215.9 63.5))
     (stroke (width 0) (type default) (color 0 0 0 0))
@@
     (stroke (width 0) (type default) (color 0 0 0 0))
   )
+  (wire (pts (xy 152.4 100.33) (xy 152.4 101.6))
+    (stroke (width 0) (type default) (color 0 0 0 0))
+  )
   (wire (pts (xy 149.86 96.52) (xy 162.56 96.52))
     (stroke (width 0) (type default) (color 0 0 0 0))
@@
     (stroke (width 0) (type default) (color 0 0 0 0))
   )
+  (wire (pts (xy 162.56 100.33) (xy 162.56 101.6))
+    (stroke (width 0) (type default) (color 0 0 0 0))
+  )
   (wire (pts (xy 226.06 96.52) (xy 228.6 96.52))
     (stroke (width 0) (type default) (color 0 0 0 0))
@@
   )
   (wire (pts (xy 190.5 50.8) (xy 190.5 63.5))
+    (stroke (width 0) (type default) (color 0 0 0 0))
+  )
+  (wire (pts (xy 203.2 100.33) (xy 203.2 101.6))
     (stroke (width 0) (type default) (color 0 0 0 0))
   )
@@
   (symbol (lib_id "Switch:SW_SPST") (at 220.98 101.6 0) (unit 1)
     (in_bom yes) (on_board yes) (fields_autoplaced)
-    (property "Reference" "SW35" (id 0) (at 220.98 95.9825 0))
-    (property "Value" "SW_SPST" (id 1) (at 220.98 98.7576 0))
+    (property "Reference" "SW35" (id 0) (at 220.98 96.2492 0))
+    (property "Value" "SW_SPST" (id 1) (at 220.98 98.7861 0))
     (property "Footprint" "keebio:MX-Alps-Choc-1U-NoLED" (id 2) (at 220.98 101.6 0)
       (effects (font (size 1.27 1.27)) hide)
@@
     )
     (property "Datasheet" "~" (id 3) (at 175.26 67.31 0)
+      (effects (font (size 1.27 1.27)) hide)
+    )
+    (pin "1")
+    (pin "2")
+  )
+  (symbol (lib_id "Switch:SW_SPST") (at 208.28 100.33 0) (unit 1)
+    (in_bom yes) (on_board yes) (fields_autoplaced)
+    (property "Reference" "SW37" (id 0) (at 208.28 94.9792 0))
+    (property "Value" "SW_SPST" (id 1) (at 208.28 97.5161 0))
+    (property "Footprint" "keebio:MX-Alps-Choc-2U" (id 2) (at 208.28 100.33 0)
+      (effects (font (size 1.27 1.27)) hide)
+    )
+    (property "Datasheet" "~" (id 3) (at 208.28 100.33 0)
       (effects (font (size 1.27 1.27)) hide)
     )
@@
     (pin "2")
   )
+  (symbol (lib_id "Switch:SW_SPST") (at 157.48 100.33 0) (unit 1)
+    (in_bom yes) (on_board yes) (fields_autoplaced)
+    (property "Reference" "SW36" (id 0) (at 157.48 94.9792 0))
+    (property "Value" "SW_SPST" (id 1) (at 157.48 97.5161 0))
+    (property "Footprint" "keebio:MX-Alps-Choc-2U" (id 2) (at 157.48 100.33 0)
+      (effects (font (size 1.27 1.27)) hide)
+    )
+    (property "Datasheet" "~" (id 3) (at 157.48 100.33 0)
+      (effects (font (size 1.27 1.27)) hide)
+    )
+    (pin "1")
+    (pin "2")
+  )
   (symbol (lib_id "Switch:SW_SPST") (at 144.78 101.6 0) (unit 1)
     (in_bom yes) (on_board yes) (fields_autoplaced)
@@
       (reference "SW35") (unit 1) (value "SW_SPST") (footprint "keebio:MX-Alps-Choc-1U-NoLED")
     )
+    (path "/efd9dcb5-02b4-4da1-9200-ec0e18dda701"
+      (reference "SW36") (unit 1) (value "SW_SPST") (footprint "keebio:MX-Alps-Choc-2U")
+    )
+    (path "/8566c05b-ea94-45b6-ae2d-b3d013af9086"
+      (reference "SW37") (unit 1) (value "SW_SPST") (footprint "keebio:MX-Alps-Choc-2U")
+    )
     (path "/fb249d71-7c05-4aff-be9f-9b3e041b0f8d"

Commit message: v0.1.3 was bad
This reverts commit 27f9da0c8f8c043d86356701b4d41a0e5f33df05.
Parts:
- removed SW36, SW37: SW_SPST, keebio:MX-Alps-Choc-2U, symbol Switch:SW_SPST
Changed lines of the file:
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@@
   (title_block
     (title "OK35")
-    (date "2022-03-06")
-    (rev "0.1.3")
+    (date "2022-02-21")
+    (rev "0.1.1")
     (company "moth.monster")
   )
@@
   (junction (at 200.66 109.22) (diameter 0) (color 0 0 0 0)
   )
-  (junction (at 162.56 101.6) (diameter 0) (color 0 0 0 0)
-  )
   (junction (at 200.66 71.12) (diameter 0) (color 0 0 0 0)
   )
@@
   (junction (at 226.06 109.22) (diameter 0) (color 0 0 0 0)
   )
-  (junction (at 203.2 100.33) (diameter 0) (color 0 0 0 0)
-  )
   (junction (at 190.5 88.9) (diameter 0) (color 0 0 0 0)
   )
@@
   (junction (at 187.96 83.82) (diameter 0) (color 0 0 0 0)
   )
-  (junction (at 213.36 101.6) (diameter 0) (color 0 0 0 0)
-  )
   (junction (at 215.9 63.5) (diameter 0) (color 0 0 0 0)
   )
-  (junction (at 152.4 100.33) (diameter 0) (color 0 0 0 0)
-  )
   (junction (at 190.5 76.2) (diameter 0) (color 0 0 0 0)
   )
@@
     (stroke (width 0) (type default) (color 0 0 0 0))
   )
-  (wire (pts (xy 152.4 88.9) (xy 152.4 100.33))
+  (wire (pts (xy 152.4 88.9) (xy 152.4 101.6))
     (stroke (width 0) (type default) (color 0 0 0 0))
   )
@@
     (stroke (width 0) (type default) (color 0 0 0 0))
   )
+  (wire (pts (xy 139.7 88.9) (xy 139.7 101.6))
+    (stroke (width 0) (type default) (color 0 0 0 0))
+  )
   (wire (pts (xy 190.5 88.9) (xy 190.5 101.6))
     (stroke (width 0) (type default) (color 0 0 0 0))
   )
-  (wire (pts (xy 139.7 88.9) (xy 139.7 101.6))
-    (stroke (width 0) (type default) (color 0 0 0 0))
-  )
   (wire (pts (xy 200.66 83.82) (xy 213.36 83.82))
     (stroke (width 0) (type default) (color 0 0 0 0))
@@
     (stroke (width 0) (type default) (color 0 0 0 0))
   )
-  (wire (pts (xy 203.2 88.9) (xy 203.2 100.33))
+  (wire (pts (xy 203.2 88.9) (xy 203.2 101.6))
     (stroke (width 0) (type default) (color 0 0 0 0))
   )
@@
     (stroke (width 0) (type default) (color 0 0 0 0))
   )
-  (wire (pts (xy 213.36 100.33) (xy 213.36 101.6))
-    (stroke (width 0) (type default) (color 0 0 0 0))
-  )
   (wire (pts (xy 215.9 50.8) (xy 215.9 63.5))
     (stroke (width 0) (type default) (color 0 0 0 0))
@@
     (stroke (width 0) (type default) (color 0 0 0 0))
   )
-  (wire (pts (xy 152.4 100.33) (xy 152.4 101.6))
-    (stroke (width 0) (type default) (color 0 0 0 0))
-  )
   (wire (pts (xy 149.86 96.52) (xy 162.56 96.52))
     (stroke (width 0) (type default) (color 0 0 0 0))
@@
     (stroke (width 0) (type default) (color 0 0 0 0))
   )
-  (wire (pts (xy 162.56 100.33) (xy 162.56 101.6))
-    (stroke (width 0) (type default) (color 0 0 0 0))
-  )
   (wire (pts (xy 226.06 96.52) (xy 228.6 96.52))
     (stroke (width 0) (type default) (color 0 0 0 0))
@@
   )
   (wire (pts (xy 190.5 50.8) (xy 190.5 63.5))
-    (stroke (width 0) (type default) (color 0 0 0 0))
-  )
-  (wire (pts (xy 203.2 100.33) (xy 203.2 101.6))
     (stroke (width 0) (type default) (color 0 0 0 0))
   )
@@
   (symbol (lib_id "Switch:SW_SPST") (at 220.98 101.6 0) (unit 1)
     (in_bom yes) (on_board yes) (fields_autoplaced)
-    (property "Reference" "SW35" (id 0) (at 220.98 96.2492 0))
-    (property "Value" "SW_SPST" (id 1) (at 220.98 98.7861 0))
+    (property "Reference" "SW35" (id 0) (at 220.98 95.9825 0))
+    (property "Value" "SW_SPST" (id 1) (at 220.98 98.7576 0))
     (property "Footprint" "keebio:MX-Alps-Choc-1U-NoLED" (id 2) (at 220.98 101.6 0)
       (effects (font (size 1.27 1.27)) hide)
@@
     )
     (property "Datasheet" "~" (id 3) (at 175.26 67.31 0)
-      (effects (font (size 1.27 1.27)) hide)
-    )
-    (pin "1")
-    (pin "2")
-  )
-  (symbol (lib_id "Switch:SW_SPST") (at 208.28 100.33 0) (unit 1)
-    (in_bom yes) (on_board yes) (fields_autoplaced)
-    (property "Reference" "SW37" (id 0) (at 208.28 94.9792 0))
-    (property "Value" "SW_SPST" (id 1) (at 208.28 97.5161 0))
-    (property "Footprint" "keebio:MX-Alps-Choc-2U" (id 2) (at 208.28 100.33 0)
-      (effects (font (size 1.27 1.27)) hide)
-    )
-    (property "Datasheet" "~" (id 3) (at 208.28 100.33 0)
       (effects (font (size 1.27 1.27)) hide)
     )
@@
     (pin "2")
   )
-  (symbol (lib_id "Switch:SW_SPST") (at 157.48 100.33 0) (unit 1)
-    (in_bom yes) (on_board yes) (fields_autoplaced)
-    (property "Reference" "SW36" (id 0) (at 157.48 94.9792 0))
-    (property "Value" "SW_SPST" (id 1) (at 157.48 97.5161 0))
-    (property "Footprint" "keebio:MX-Alps-Choc-2U" (id 2) (at 157.48 100.33 0)
-      (effects (font (size 1.27 1.27)) hide)
-    )
-    (property "Datasheet" "~" (id 3) (at 157.48 100.33 0)
-      (effects (font (size 1.27 1.27)) hide)
-    )
-    (pin "1")
-    (pin "2")
-  )
   (symbol (lib_id "Switch:SW_SPST") (at 144.78 101.6 0) (unit 1)
     (in_bom yes) (on_board yes) (fields_autoplaced)
@@
       (reference "SW35") (unit 1) (value "SW_SPST") (footprint "keebio:MX-Alps-Choc-1U-NoLED")
     )
-    (path "/efd9dcb5-02b4-4da1-9200-ec0e18dda701"
-      (reference "SW36") (unit 1) (value "SW_SPST") (footprint "keebio:MX-Alps-Choc-2U")
-    )
-    (path "/8566c05b-ea94-45b6-ae2d-b3d013af9086"
-      (reference "SW37") (unit 1) (value "SW_SPST") (footprint "keebio:MX-Alps-Choc-2U")
-    )
     (path "/fb249d71-7c05-4aff-be9f-9b3e041b0f8d"

Commit message: v0.1.2 finalized public release
Other:
- title: OK35 -> OK35 Public Release
Changed lines of the file:
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@@
   (paper "A4")
   (title_block
-    (title "OK35")
-    (date "2022-02-21")
-    (rev "0.1.1")
+    (title "OK35 Public Release")
+    (date "2022-03-10")
+    (rev "0.1.2")
     (company "moth.monster")
   )

Commit message: number mistake
Parts:
- R1, R2: value 2K2 -> 10k
Changed lines of the file:
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@@
       (effects (font (size 1.27 1.27)) (justify left) hide)
     )
-    (property "Value" "2K2" (id 1) (at 101.6 68.58 90))
+    (property "Value" "10k" (id 1) (at 101.6 68.58 90))
     (property "Footprint" "Resistor_THT:R_Axial_DIN0207_L6.3mm_D2.5mm_P7.62mm_Horizontal" (id 2) (at 101.6 70.358 90)
       (effects (font (size 1.27 1.27)) hide)
@@
       (effects (font (size 1.27 1.27)) (justify left) hide)
     )
-    (property "Value" "2K2" (id 1) (at 101.6 72.39 90))
+    (property "Value" "10k" (id 1) (at 101.6 72.39 90))
     (property "Footprint" "Resistor_THT:R_Axial_DIN0207_L6.3mm_D2.5mm_P7.62mm_Horizontal" (id 2) (at 101.6 74.168 90)
       (effects (font (size 1.27 1.27)) hide)
@@
     )
     (path "/37e9bfa6-9f52-4e15-b12d-0781db7a2c82"
-      (reference "R1") (unit 1) (value "2K2") (footprint "Resistor_THT:R_Axial_DIN0207_L6.3mm_D2.5mm_P7.62mm_Horizontal")
+      (reference "R1") (unit 1) (value "10k") (footprint "Resistor_THT:R_Axial_DIN0207_L6.3mm_D2.5mm_P7.62mm_Horizontal")
     )
     (path "/88b31a51-f886-4b2b-b511-2e3ab761a629"
-      (reference "R2") (unit 1) (value "2K2") (footprint "Resistor_THT:R_Axial_DIN0207_L6.3mm_D2.5mm_P7.62mm_Horizontal")
+      (reference "R2") (unit 1) (value "10k") (footprint "Resistor_THT:R_Axial_DIN0207_L6.3mm_D2.5mm_P7.62mm_Horizontal")
     )
     (path "/c1d4cce4-9fc8-49e7-8c15-24df5623c3cb"
